File: Elekit2.0v1.kicad_sch (KiCad schematic)
At the start: 124 parts, among them J1 Screw_Terminal_01x02, J10 Conn_01x03_Male, J11 DS18B20 temperature sensor, J12 Conn_01x01_Male, J13 Conn_01x01_Male, J2 Screw_Terminal_01x02, J3 Screw_Terminal_01x02, J4 Screw_Terminal_01x02, J5 Conn_01x03_Male, J6 Conn_01x06_Male, J7 Conn_01x08, J8 Conn_01x08, J9 Conn_01x03_Male, Q1 2N7002, Q2 2N7002, Q3 2N7002, SW1 SW_Push, SW2 SW_Push, SW3 SW_Push, SW4 SW_Push, SW5 SW_Push, SW6 SW_Push, U1 MINI_5PTP, U10 TS-1187A-B-A-B, U11 DHT11, U12 DRV8870DDA, U13 74HC165, U15 DRV8870DDA, U2 MY-2032-12, U3 L7805, U4 MY-2032-12, U5 SRV05-4-P-T7, U6 74HC595, U7 ME6211C33M5G-N, U8 TS-1187A-B-A-B, U9 ESP32-C3-WROOM-02-N4(4MB)

Commit message: Create first complete version
Parts:
- removed C24: 0.1u 50V, Capacitor_SMD:C_0402_1005Metric, symbol Device:C_Small
- removed C25: 1u, Capacitor_SMD:C_0805_2012Metric, symbol Device:C_Small
- removed C26: C_Polarized, Capacitor_THT:CP_Radial_D5.0mm_P2.00mm, symbol Device:C_Polarized
- removed JP10, JP11, JP12, JP13: Servo1, Jumper:SolderJumper-2_P1.3mm_Open_RoundedPad1.0x1.5mm, symbol Jumper:SolderJumper_2_Open
- removed JP14: Latch control, Jumper:SolderJumper-2_P1.3mm_Open_RoundedPad1.0x1.5mm, symbol Jumper:SolderJumper_2_Open
- removed R20, R23, R24, R25, R26: 1k, Resistor_SMD:R_0402_1005Metric, symbol Device:R
- removed R22, R28, R29, R30, R33: 10k, Resistor_SMD:R_0402_1005Metric, symbol Device:R
- removed U13: 74HC165, 0_JLCPCB_Footprints:SOIC-16_L9.9-W3.9-P1.27-LS6.0-BL, symbol 74xx:74HC165
- added C10: 1u, Capacitor_SMD:C_0805_2012Metric, symbol Device:C_Small
- C12, C13, C14, C15, C16, C17, C18, C20, C21, C22, C5, C6, C7: value 0.1u 50V -> 0.1u; footprint Capacitor_SMD:C_0402_1005Metric -> Capacitor_SMD:C_0805_2012Metric; LCSC C307331 -> C28233
- DS1: footprint SnapEDA Library:LCD_RC1602B-BIW-CSV -> Display:WC1602A
- JP3: value H-Bridge -> Latch control
- JP4: value PWR LED -> Power LED
- R10, R13, R14, R3, R5, R8, R9: footprint Resistor_SMD:R_0402_1005Metric -> Resistor_SMD:R_0805_2012Metric; LCSC C11702 -> C17513
- R12, R15, R17: footprint Resistor_SMD:R_0402_1005Metric -> Resistor_SMD:R_1206_3216Metric; LCSC C25744 -> C4410
- R18, R6: footprint Resistor_SMD:R_0402_1005Metric -> Resistor_SMD:R_0805_2012Metric; LCSC C25744 -> C17414
- R4: value 1k -> 10k; footprint Resistor_SMD:R_0402_1005Metric -> Resistor_SMD:R_0805_2012Metric; LCSC C11702 -> C17414
Connections:
- net BTN2 is gone; now on net GND: C16.1
- net BTN3 is gone; now on net GND: C17.1
- net BTN4 is gone; now on net GND: C20.1
- net BTN5 is gone; now on net GND: C21.1
- net +3.3V: now also U12.4 (VREF), U15.4 (VREF); no longer JP3.1 (A)
- net A1: now also J2.1 (Pin_1); no longer J2.2 (Pin_2)
- net A1_c: no longer J7.7 (Pin_7), U9.5 (IO6)
- net A2: now also J2.2 (Pin_2); no longer J2.1 (Pin_1)
- net A2_C: no longer J7.8 (Pin_8), U9.6 (IO7)
- net B1: now also J3.1 (Pin_1); no longer J3.2 (Pin_2)
- net B1_c: no longer J7.5 (Pin_5), U9.3 (IO4)
- net B2: now also J3.2 (Pin_2); no longer J3.1 (Pin_1)
- net B2_C: no longer J7.6 (Pin_6), U9.4 (IO5)
- net GND: now also C14.1, SW2.1, SW3.1, SW4.1, SW5.1, SW6.1, C10.2; no longer C14.2
- net GPIO2: no longer R10.2
- net RX: no longer U6.14 (SER)
- net VBUS: no longer C14.1, C16.2, C17.2, C20.2, C21.2, SW2.1, SW3.1, SW4.1, SW5.1, SW6.1
- net at SW6.2: now also C21.2
- net at SW4.2: now also C17.2
- net at SW5.2: now also C20.2
- net at SW2.2: now also C14.2
- net at SW3.2: now also C16.2
- net BTN1 renamed BTN
- net BTN: now also C10.1
- net CLK1 renamed GPIO10
- net CLK2: no longer names the net of U6.11 (SRCLK), U6.12 (RCLK)
- net CLK2: no longer J7.4 (Pin_4), U9.15 (IO3)
- removed net H-BRIDGE_PWR: JP3.2 (B), U12.4 (VREF), U15.4 (VREF)
- net Latch control: no longer names the net of R5.2
- net Latch control: now also JP3.1 (A)
- net SERVO1_c renamed GPIO5
- net GPIO5: now also J7.6 (Pin_6), R10.2, U9.4 (IO5)
- net SERVO2_c renamed GPIO6
- net GPIO6: now also J7.7 (Pin_7), U9.5 (IO6)
- new net GPIO3: J7.4 (Pin_4), U9.15 (IO3)
- new net GPIO4: J7.5 (Pin_5), JP3.2 (B), U9.3 (IO4)
- new net GPIO7: J7.8 (Pin_8), U9.6 (IO7)
Other:
- moved on the sheet: C13, C15, C4, C5, D2, U10, U3, U8
