File: Elekit2.0.kicad_sch (KiCad schematic)
At the start: 124 parts, among them J1 Screw_Terminal_01x02, J10 Conn_01x03_Male, J11 DS18B20 temperature sensor, J12 Conn_01x01_Male, J13 Conn_01x01_Male, J2 Screw_Terminal_01x02, J3 Screw_Terminal_01x02, J4 Screw_Terminal_01x02, J5 Conn_01x03_Male, J6 Conn_01x06_Male, J7 Conn_01x08, J8 Conn_01x08, J9 Conn_01x03_Male, Q1 2N7002, Q2 2N7002, Q3 2N7002, SW1 SW_Push, SW2 SW_Push, SW3 SW_Push, SW4 SW_Push, SW5 SW_Push, SW6 SW_Push, U1 MINI_5PTP, U10 TS-1187A-B-A-B, U11 DHT11, U12 DRV8870DDA, U13 74HC165, U15 DRV8870DDA, U2 MY-2032-12, U3 L7805, U4 MY-2032-12, U5 SRV05-4-P-T7, U6 74HC595, U7 ME6211C33M5G-N, U8 TS-1187A-B-A-B, U9 ESP32-C3-WROOM-02-N4(4MB)

Commit message: production updates
Parts:
- removed C3: 4.7n, Capacitor_SMD:C_0805_2012Metric, symbol Device:C_Small
- removed J7, J8: Conn_01x08, Connector_PinHeader_2.54mm:PinHeader_1x08_P2.54mm_Vertical, symbol Connector_Generic:Conn_01x08
- removed R1: 1M, Resistor_SMD:R_1206_3216Metric, symbol Device:R
- added J7: Conn_01x04, Connector_PinSocket_2.54mm:PinSocket_1x04_P2.54mm_Vertical, symbol Connector_Generic:Conn_01x04
Connections:
- net +3.3V: now also J7.4 (Pin_4)
- net GND: now also J7.1 (Pin_1)
- net GPIO0: now also J7.2 (Pin_2)
- net GPIO1: now also J7.3 (Pin_3)
- now unconnected: U1.6, U1.7, U1.8, U1.9
Other:
- moved on the sheet: LOGO1, RV1
